File: eink-kicad/eink.sch (KiCad schematic (older format))
At the start: 79 parts, among them J1 0R, P1 CONN_1, P10 CONN_1, P11 CONN_1, P12 CONN_1, P13 CONN_1, P14 CONN_1, P15 CONN_1, P16 CONN_1, P17 CONN_1, P18 CONN_1, P19 CONN_1, P2 CONN_1, P20 CONN_1, P21 CONN_1, P22 CONN_1, P23 CONN_1, P24 CONN_1, P25 CONN_1, P26 CONN_1, P27 CONN_1, P28 CONN_1, P29 CONN_1, P3 CONN_1, P30 CONN_1, P31 CONN_1, P32 CONN_1, P33 CONN_1, P34 CONN_1, P35 CONN_1, P36 CONN_1, P37 CONN_1, P38 CONN_1, P39 CONN_1, P4 CONN_1, P40 CONN_1, P41 CONN_1, P42 CONN_1, P43 CONN_1, P5 CONN_1, P6 CONN_1, P7 CONN_1, P8 CONN_1, P9 CONN_1, Q1 MOS_P, U1 LT1945, U2 78L15, U3 79L15, U4 LM358, U5 ED060SC4V2-FPC

Commit message: Terminate the LM358's other op-amp.
Parts:
- added unit 2 of U4
Connections:
- wire segments 124 -> 130
Changed lines of the file:
@@
 Sheet 1 1
 Title ""
-Date "24 sep 2015"
+Date "5 oct 2015"
 Rev ""
 Comp ""
@@
 	1    0    0    -1
 $EndComp
+$Comp
+L LM358 U4
+U 2 1 5612EA1F
+P 5050 6450
+F 0 "U4" H 5000 6650 60  0000 L CNN
+F 1 "LM358" H 5000 6200 60  0000 L CNN
+F 2 "" H 5050 6450 60  0000 C CNN
+F 3 "" H 5050 6450 60  0000 C CNN
+	2    5050 6450
+	1    0    0    -1
+$EndComp
+Wire Wire Line
+	4550 6550 4550 7250
+Wire Wire Line
+	4550 7250 5550 7250
+Wire Wire Line
+	5550 7250 5550 6450
+Text Label 4950 7100 0    60   ~ 0
+-15V
+Text Label 4950 5750 0    60   ~ 0
++15V
+Wire Wire Line
+	4550 6350 4050 6350
+Text Label 4050 6350 0    60   ~ 0
+GND
+Wire Wire Line
+	4950 6050 4950 5750
+Wire Wire Line
+	4950 6850 4950 7100
 $EndSCHEMATC

Commit message: Fix FPC connector pinout and turn it around to face edge.
Parts:
- removed P29, P31, P43, P8: CONN_1, SIL-1, symbol CONN_1
- renumbered P30 to P29, P32 to P30, P33 to P31, P34 to P32, P35 to P33, P36 to P34, P37 to P35, P38 to P36, P39 to P37, P40 to P38, P41 to P39, P42 to P40, U4 to U2, U2 to U3, U3 to U4
Connections:
- net labels removed: GVEE
Changed lines of the file:
@@
 Sheet 1 1
 Title ""
-Date "5 oct 2015"
+Date "17 oct 2015"
 Rev ""
 Comp ""
@@
 $EndComp
 $Comp
-L 78L15 U2
+L 78L15 U3
 U 1 1 55E24930
 P 6400 3750
-F 0 "U2" H 6550 3554 60  0000 C CNN
+F 0 "U3" H 6550 3554 60  0000 C CNN
 F 1 "78L15" H 6400 3950 60  0000 C CNN
 F 2 "78LxxA" H 6400 4050 60  0000 C CNN
@@
 $EndComp
 $Comp
-L 79L15 U3
+L 79L15 U4
 U 1 1 55E2493F
 P 6800 2300
-F 0 "U3" H 6950 2104 60  0000 C CNN
+F 0 "U4" H 6950 2104 60  0000 C CNN
 F 1 "79L15" H 6800 2500 60  0000 C CNN
 F 2 "79LxxA" H 6800 2600 60  0000 C CNN
@@
 1
 $Comp
-L LM358 U4
-U 1 1 55E2882E
+L LM358 U2
+U 2 1 55E2882E
 P 8200 1400
-F 0 "U4" H 8150 1600 60  0000 L CNN
+F 0 "U2" H 8150 1600 60  0000 L CNN
 F 1 "LM358" H 8150 1150 60  0000 L CNN
 F 2 "MSOP_8" H 8300 1000 60  0000 C CNN
 F 3 "" H 8200 1400 60  0000 C CNN
-	1    8200 1400
+	2    8200 1400
 	1    0    0    -1
 $EndComp
@@
 $EndComp
 $Comp
-L CONN_1 P39
+L CONN_1 P37
 U 1 1 55F8A184
 P 8900 5700
-F 0 "P39" H 8980 5700 40  0000 L CNN
+F 0 "P37" H 8980 5700 40  0000 L CNN
 F 1 "CONN_1" H 8900 5755 30  0001 C CNN
 F 2 "SIL-1" H 9200 5700 60  0000 C CNN
@@
 $EndComp
 $Comp
-L CONN_1 P38
+L CONN_1 P36
 U 1 1 55F8A601
 P 8900 5600
-F 0 "P38" H 8980 5600 40  0000 L CNN
+F 0 "P36" H 8980 5600 40  0000 L CNN
 F 1 "CONN_1" H 8900 5655 30  0001 C CNN
 F 2 "SIL-1" H 9200 5600 60  0000 C CNN
@@
 $EndComp
 $Comp
-L CONN_1 P37
+L CONN_1 P35
 U 1 1 55F8A607
 P 8900 5500
-F 0 "P37" H 8980 5500 40  0000 L CNN
+F 0 "P35" H 8980 5500 40  0000 L CNN
 F 1 "CONN_1" H 8900 5555 30  0001 C CNN
 F 2 "SIL-1" H 9200 5500 60  0000 C CNN
@@
 $EndComp
 $Comp
-L CONN_1 P34
+L CONN_1 P32
 U 1 1 55F8A60D
 P 8900 5000
-F 0 "P34" H 8980 5000 40  0000 L CNN
+F 0 "P32" H 8980 5000 40  0000 L CNN
 F 1 "CONN_1" H 8900 5055 30  0001 C CNN
 F 2 "SIL-1" H 9200 5000 60  0000 C CNN
@@
 $EndComp
 $Comp
-L CONN_1 P33
+L CONN_1 P31
 U 1 1 55F959FC
 P 8900 4900
-F 0 "P33" H 8980 4900 40  0000 L CNN
+F 0 "P31" H 8980 4900 40  0000 L CNN
 F 1 "CONN_1" H 8900 4955 30  0001 C CNN
 F 2 "SIL-1" H 9200 4900 60  0000 C CNN
@@
 $EndComp
 $Comp
-L CONN_1 P32
+L CONN_1 P30
 U 1 1 55F95A02
 P 8900 4800
-F 0 "P32" H 8980 4800 40  0000 L CNN
+F 0 "P30" H 8980 4800 40  0000 L CNN
 F 1 "CONN_1" H 8900 4855 30  0001 C CNN
 F 2 "SIL-1" H 9200 4800 60  0000 C CNN
@@
 $EndComp
 $Comp
-L CONN_1 P42
+L CONN_1 P40
 U 1 1 55F95A14
 P 8900 6200
-F 0 "P42" H 8980 6200 40  0000 L CNN
+F 0 "P40" H 8980 6200 40  0000 L CNN
 F 1 "CONN_1" H 8900 6255 30  0001 C CNN
 F 2 "SIL-1" H 9200 6200 60  0000 C CNN
@@
 $EndComp
 $Comp
-L CONN_1 P35
+L CONN_1 P33
 U 1 1 55FBCA66
 P 8900 5300
-F 0 "P35" H 8980 5300 40  0000 L CNN
+F 0 "P33" H 8980 5300 40  0000 L CNN
 F 1 "CONN_1" H 8900 5355 30  0001 C CNN
 F 2 "SIL-1" H 9200 5300 60  0000 C CNN
@@
 $EndComp
 $Comp
-L CONN_1 P36
+L CONN_1 P34
 U 1 1 55FBCA6C
 P 8900 5400
-F 0 "P36" H 8980 5400 40  0000 L CNN
+F 0 "P34" H 8980 5400 40  0000 L CNN
 F 1 "CONN_1" H 8900 5455 30  0001 C CNN
 F 2 "SIL-1" H 9200 5400 60  0000 C CNN
@@
 $EndComp
 $Comp
-L CONN_1 P40
+L CONN_1 P38
 U 1 1 55FBCA72
 P 8900 5800
-F 0 "P40" H 8980 5800 40  0000 L CNN
+F 0 "P38" H 8980 5800 40  0000 L CNN
 F 1 "CONN_1" H 8900 5855 30  0001 C CNN
 F 2 "SIL-1" H 9200 5800 60  0000 C CNN
@@
 $EndComp
 $Comp
-L CONN_1 P41
+L CONN_1 P39
 U 1 1 55FBCA78
 P 8900 5900
-F 0 "P41" H 8980 5900 40  0000 L CNN
+F 0 "P39" H 8980 5900 40  0000 L CNN
 F 1 "CONN_1" H 8900 5955 30  0001 C CNN
 F 2 "SIL-1" H 9200 5900 60  0000 C CNN
@@
 	9700 4600 9050 4600
 $Comp
-L CONN_1 P31
-U 1 1 5603262A
-P 8900 4700
-F 0 "P31" H 8980 4700 40  0000 L CNN
-F 1 "CONN_1" H 8900 4755 30  0001 C CNN
-F 2 "SIL-1" H 9200 4700 60  0000 C CNN
-F 3 "" H 8900 4700 60  0000 C CNN
-	1    8900 4700
-	-1   0    0    1
-$EndComp
-$Comp
-L CONN_1 P30
+L CONN_1 P29
 U 1 1 5603263A
 P 8900 4600
-F 0 "P30" H 8980 4600 40  0000 L CNN
+F 0 "P29" H 8980 4600 40  0000 L CNN
 F 1 "CONN_1" H 8900 4655 30  0001 C CNN
 F 2 "SIL-1" H 9200 4600 60  0000 C CNN
@@
 	1    0    0    -1
 $EndComp
-$Comp
-L CONN_1 P8
-U 1 1 5603265A
-P 7450 4700
-F 0 "P8" H 7530 4700 40  0000 L CNN
-F 1 "CONN_1" H 7450 4755 30  0001 C CNN
-F 2 "SIL-1" H 7750 4700 60  0000 C CNN
-F 3 "" H 7450 4700 60  0000 C CNN
-	1    7450 4700
-	1    0    0    -1
-$EndComp
 Wire Wire Line
 	9700 2500 9050 2500
@@
 Text Label 9050 4600 0    60   ~ 0
 GVDD
-Text Label 9050 4700 0    60   ~ 0
-GVEE
 $Comp
 L CONN_1 P11
@@
 Wire Wire Line
 	8700 1400 9300 1400
-$Comp
-L CONN_1 P29
-U 1 1 56032FAA
-P 8900 4500
-F 0 "P29" H 8980 4500 40  0000 L CNN
-F 1 "CONN_1" H 8900 4555 30  0001 C CNN
-F 2 "SIL-1" H 9200 4500 60  0000 C CNN
-F 3 "" H 8900 4500 60  0000 C CNN
-	1    8900 4500
-	-1   0    0    1
-$EndComp
 Text Label 9050 4500 0    60   ~ 0
 VCOM
-$Comp
-L CONN_1 P43
-U 1 1 56033218
-P 9450 1400
-F 0 "P43" H 9530 1400 40  0000 L CNN
-F 1 "CONN_1" H 9450 1455 30  0001 C CNN
-F 2 "SIL-1" H 9750 1400 60  0000 C CNN
-F 3 "" H 9450 1400 60  0000 C CNN
-	1    9450 1400
-	1    0    0    -1
-$EndComp
 $Comp
 L CONN_1 P9
@@
 $Comp
 L PWR_FLAG #FLG016
-U 1 1 560343BB
-P 9050 4700
-F 0 "#FLG016" H 9050 4795 30  0001 C CNN
-F 1 "PWR_FLAG" H 9050 4880 30  0000 C CNN
-F 2 "" H 9050 4700 60  0000 C CNN
-F 3 "" H 9050 4700 60  0000 C CNN
-	1    9050 4700
-	1    0    0    -1
-$EndComp
-$Comp
-L PWR_FLAG #FLG017
 U 1 1 560343CB
 P 9050 4600
-F 0 "#FLG017" H 9050 4695 30  0001 C CNN
+F 0 "#FLG016" H 9050 4695 30  0001 C CNN
 F 1 "PWR_FLAG" H 9050 4780 30  0000 C CNN
 F 2 "" H 9050 4600 60  0000 C CNN
@@
 $EndComp
 $Comp
-L PWR_FLAG #FLG018
+L PWR_FLAG #FLG017
 U 1 1 560343DB
 P 9050 2500
-F 0 "#FLG018" H 9050 2595 30  0001 C CNN
+F 0 "#FLG017" H 9050 2595 30  0001 C CNN
 F 1 "PWR_FLAG" H 9050 2680 30  0000 C CNN
 F 2 "" H 9050 2500 60  0000 C CNN
@@
 $EndComp
 $Comp
-L PWR_FLAG #FLG019
+L PWR_FLAG #FLG018
 U 1 1 560343E1
 P 9050 2400
-F 0 "#FLG019" H 9050 2495 30  0001 C CNN
+F 0 "#FLG018" H 9050 2495 30  0001 C CNN
 F 1 "PWR_FLAG" H 9050 2580 30  0000 C CNN
 F 2 "" H 9050 2400 60  0000 C CNN
@@
 $EndComp
 $Comp
-L PWR_FLAG #FLG020
-U 1 1 560343EA
-P 9050 4500
-F 0 "#FLG020" H 9050 4595 30  0001 C CNN
-F 1 "PWR_FLAG" H 9050 4680 30  0000 C CNN
-F 2 "" H 9050 4500 60  0000 C CNN
-F 3 "" H 9050 4500 60  0000 C CNN
-	1    9050 4500
-	1    0    0    -1
-$EndComp
-$Comp
-L LM358 U4
-U 2 1 5612EA1F
+L LM358 U2
+U 1 1 5612EA1F
 P 5050 6450
-F 0 "U4" H 5000 6650 60  0000 L CNN
+F 0 "U2" H 5000 6650 60  0000 L CNN
 F 1 "LM358" H 5000 6200 60  0000 L CNN
 F 2 "" H 5050 6450 60  0000 C CNN
 F 3 "" H 5050 6450 60  0000 C CNN
-	2    5050 6450
+	1    5050 6450
 	1    0    0    -1
 $EndComp
@@
 Wire Wire Line
 	4950 6850 4950 7100
+Text Label 9300 1400 2    60   ~ 0
+VCOM
+Text Label 9050 4700 0    60   ~ 0
+-20V
 $EndSCHEMATC

Commit message: New version of board for new version of KiCad :)
Parts:
- removed J1: 0R, Resistor_SMD0805_HandSoldering_RevA_Date21Jun2010, symbol R
- removed P10, P11, P12, P29, P6, P7, P9: CONN_1, SIL-1, symbol CONN_1
- C1, C2, C3, C4, C5, C6, C7, C8: footprint Capacitor_SMD0805_HandSoldering_RevA_Date21Jun2010 -> Capacitors_SMD:C_0805_HandSoldering; symbol C -> C-RESCUE-eink
- C9: footprint C1 -> Capacitors_ThroughHole:C_Radial_D5_L6_P2.5; symbol CP1 -> CP1-RESCUE-eink
- D1, D2, D3: footprint Diode-Universal-SMB-SMC_Handsoldering_RevA_27July2010 -> Diodes_SMD:SMB-SMC_Universal_Handsoldering
- L1, L2: footprint SELF-WE-TPC_M -> Inductors:SELF-WE-TPC_M
- P1, P13, P14, P15, P16, P17, P18, P19, P2, P20, P21, P22, P23, P24, P25, P26, P27, P28, P3, P30, P31, P32, P33, P34, P35, P36, P37, P38, P39, P4, P40, P5: footprint SIL-1 -> Pin_Headers:Pin_Header_Straight_1x01
- Q1: footprint IRLML6402 -> eink-footprints:IRLML6402
- R1, R2, R3, R4, R5, R6, R7, R8: footprint Resistor_SMD0805_HandSoldering_RevA_Date21Jun2010 -> Resistors_SMD:R_0805_HandSoldering; symbol R -> R-RESCUE-eink
- RV1: footprint Bourns_3314G-1 -> eink-footprints:Bourns_3314G-1
- TP1, TP2, TP3, TP4, TP5, TP6: footprint SIL-1 -> Measurement_Points:Measurement_Point_Round-TH_Small
- U1: footprint MSOP10-0.5 -> Housings_SSOP:MSOP-10_3x3mm_Pitch0.5mm
- U2: footprint MSOP_8 -> Housings_SSOP:MSOP-8_3x3mm_Pitch0.65mm; symbol LM358 -> LM358-RESCUE-eink
- U2: footprint (none) -> Housings_SSOP:MSOP-8_3x3mm_Pitch0.65mm; symbol LM358 -> LM358-RESCUE-eink
- U3: footprint 78LxxA -> eink-footprints:78LxxA
- U4: footprint 79LxxA -> eink-footprints:79LxxA
- U5: footprint FH26-39S-0.3SHW -> eink-footprints:FH26-39S-0.3SHW
Connections:
- net labels removed: GVDD, VDD
- wire segments 130 -> 133

Commit message: Revision 2 of board with shift registers.
Parts:
- removed P1, P14, P16, P17, P18, P19, P20, P21, P22, P23, P24, P25, P26, P27, P28, P3, P30, P31, P32, P33, P34, P35, P36, P38, P39, P4, P40, P5: CONN_1, Pin_Headers:Pin_Header_Straight_1x01, symbol CONN_1
- removed TP1, TP2, TP3, TP4, TP5, TP6: CONN_1, Measurement_Points:Measurement_Point_Round-TH_Small, symbol CONN_1
- added P10, P2, P3, P5, P6: CONN_01X01, Pin_Headers:Pin_Header_Straight_1x01, symbol CONN_01X01
- added SW1, SW10, SW11, SW12, SW13, SW2, SW3, SW4, SW5, SW6, SW7, SW8, SW9: SW_SPDT_Small, Pin_Headers:Pin_Header_Straight_1x03, symbol SW_SPDT_Small
- added U3, U4: 74HC595, Housings_DIP:DIP-16_W7.62mm_LongPads, symbol 74HC595
- added W1, W2, W3, W4, W5, W6, W7, W8: TEST_1P, Measurement_Points:Measurement_Point_Round-TH_Big, symbol TEST_1P
- D1, D2, D3: value DIODESCH -> D_Schottky; symbol DIODESCH -> D_Schottky
- RV1: footprint eink-footprints:Bourns_3314G-1 -> eink-footprints:Bourns_3314G-1-biggerpads
- U7: renamed from U5; footprint eink-footprints:FH26-39S-0.3SHW -> eink-footprints:FH26-39S-0.3SHW-biggerpads
- renumbered P2 to P1, P13 to P7, P15 to P8, P37 to P9, U3 to U5, U4 to U6
Connections:
- net labels added: CE1, CE2, LATCH, RL, SHR, SRCLK, SRDATA, VCC, ~SRCLR~, ~SROE~
- net labels removed: P10, P9
- wire segments 133 -> 141
- no-connect marks 0 -> 1
Other:
- moved on the sheet: P1, P9, U2A
