File: pcb/eink.sch (KiCad schematic (older format))
At the start: 61 parts, among them P1 CONN_1, P10 CONN_01X01, P2 CONN_01X01, P3 CONN_01X01, P5 CONN_01X01, P6 CONN_01X01, P7 CONN_1, P8 CONN_1, P9 CONN_1, Q1 MOS_P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

Commit message: Resave kicad files with a new (?) version, rescued trimpot part.
Parts:
- RV1: symbol POT -> POT-RESCUE-eink
Changed lines of the file:
@@
 LIBS:eink-lib
 LIBS:eink-cache
-EELAYER 25 0
+EELAYER 26 0
 EELAYER END
 $Descr A4 11693 8268
@@
 NOTE: 7xL15 output components - es: 10K, 4.7uF; sm: 39K? 3.9K?, 0.1uF?
 $Comp
-L POT RV1
+L POT-RESCUE-eink RV1
 U 1 1 55F882B6
 P 7300 1300

Commit message: Update revision on schematic.
Changed lines of the file:
@@
 ED060SC4 power and breakout board
 Text Label 10650 7650 0    60   ~ 0
-1
+2
 $Comp
 L LM358-RESCUE-eink U2
